Commit message: major refactoring and usability

File: gym_duckietown3/assets/urdf/robot/robot_clean_big.urdf (robot description, URDF)
Before this commit: robot mybot, 7 links, 6 joints
Links:
- link caster_wheel: mass 10 -> 1
- link chassis: mass 50 -> 5
- link left_wheel: mass 10 -> 1
- link right_wheel: mass 10 -> 1
